File: Proyecto/MóduloElectrónico/Sensing probe/Sensing probe.kicad_pcb (KiCad board)
At the start: 2 copper layers, 95.2 x 38.1 mm, 44 parts, among them J1 Conn_01x02, J2 Conn_01x02, J3 Conn_01x03_Pin, J4 Conn_01x02, J5 Conn_01x02, U1 CA3140, U2 LM324, U4 CA3140, U5 LM324

Commit message: Update sensing board
Parts:
- removed the G*** at (119.4, 108.0)
- added D1: 1N4007, Diode_THT:D_DO-34_SOD68_P2.54mm_Vertical_AnodeUp, F.Cu at (118.1, 104.8)
- added J6: Conn_01x03_Pin, Connector_PinHeader_2.54mm:PinHeader_1x03_P2.54mm_Vertical, F.Cu at (205.7, 111.1)
- added K1: HFD23, JohnsCustomLibrary:HFD23, F.Cu at (120.7, 113.1)
- added Q1: Q_NPN_EBC, Package_TO_SOT_THT:TO-92, F.Cu at (120.7, 101.6)
Connections:
- U3 pad 16: unconnected-(U3-TX1-Pad16) -> /TX
- U3 pad 25: unconnected-(U3-D7-Pad25) -> /RELAY
Routing:
- net /RELAY: track 0.00 -> 78.8 mm
- net /TX: track 0.00 -> 45.3 mm
- net GND: track 215.3 -> 231.6 mm
- net +5V: track 157.3 -> 172.9 mm
- net Net-(D1-K): track 0.00 -> 11.5 mm
- net /TEMP: track 32.0 -> 40.8 mm
- net /REF: track 140.6 -> 144.9 mm
- net /PULSE: track 76.8 -> 79.0 mm
- added copper zone on B.Cu, net GND
- added copper zone on F.Cu, net GND

Commit message: Desconector de sensor de conductividad
Parts:
- added K2: HFD23, JohnsCustomLibrary:HFD23, F.Cu at (145.4, 121.9)
- moved G*** 76.1 mm to (208.3, 108.0), turned to 90 degrees
- moved J1 32.1 mm to (135.9, 123.8), turned to -90 degrees
- moved J6 7.88 mm to (200.9, 117.3), turned to 180 degrees
- moved J5 6.01 mm to (194.8, 112.3), turned to 90 degrees
- moved U1 3.81 mm to (141.0, 108.0)
- moved C2 3.81 mm to (146.0, 104.8)
- moved C5 1.92 mm to (200.0, 122.0)
- moved R19 0.64 mm to (197.4, 115.3)
Connections:
- J1 pad 1: /SIGNAL -> /ELECTRODE_B
- J1 pad 2: /COND_READ -> /ELECTRODE_A
- K1 pad 11: unconnected-(K1-Pad11)_1 -> /ELECTRODE_A
- K1 pad 13: unconnected-(K1-Pad13) -> /SIGNAL
Routing:
- net Net-(D1-K): track 11.5 -> 43.6 mm
- net /ELECTRODE_B: track 0.00 -> 21.5 mm
- net /TURB: track 89.4 -> 68.2 mm
- net /ELECTRODE_A: track 0.00 -> 18.2 mm
- net GND: track 231.6 -> 214.5 mm
- net /COND_READ: track 22.8 -> 35.7 mm
- net /SIGNAL: track 76.4 -> 86.9 mm
- net /PH: track 52.2 -> 43.1 mm
- net +5V: track 172.9 -> 180.4 mm
- net Net-(J2-Pin_1): track 30.1 -> 37.0 mm
- net Net-(U1--): track 22.4 -> 16.8 mm
- net Net-(J5-Pin_1): track 20.7 -> 15.3 mm
- net /REF: track 144.9 -> 149.7 mm
- net /TX: track 45.3 -> 41.4 mm
- net /DO: track 36.1 -> 39.7 mm
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
Commit message: Add files via upload
Parts:
- added D2: 1N4007, Diode_THT:D_DO-34_SOD68_P2.54mm_Vertical_AnodeUp, F.Cu at (153.3, 124.2)
- moved G*** 0.36 mm to (207.9, 107.9)
Routing:
- net Net-(D1-K): track 43.6 -> 55.1 mm
- net GND: track 214.5 -> 225.9 mm
- net +5V: track 180.4 -> 179.4 mm

Commit message: Branch alternativo
Parts:
- added J5: Conn_01x03_Pin, Connector_PinHeader_2.54mm:PinHeader_1x03_P2.54mm_Vertical, F.Cu at (186.1, 114.6)
- added R22: 1K, Resistor_THT:R_Axial_DIN0204_L3.6mm_D1.6mm_P2.54mm_Vertical, F.Cu at (117.3, 105.2)
- added R23: 10K, Resistor_THT:R_Axial_DIN0204_L3.6mm_D1.6mm_P2.54mm_Vertical, F.Cu at (162.3, 111.6)
- added R24: 15K, Resistor_THT:R_Axial_DIN0204_L3.6mm_D1.6mm_P2.54mm_Vertical, F.Cu at (160.1, 114.0)
- R2: value 10K -> 3.3K
- R20: value 10K -> 15K
- R5: value 50K -> 33K
- moved R20 13.2 mm to (178.8, 117.3)
- moved R10 7.88 mm to (145.0, 92.5), turned to 180 degrees
- moved Q1 3.75 mm to (117.6, 99.4)
- moved R19 3.30 mm to (194.1, 115.3), turned to 0 degrees
- moved D1 2.05 mm to (118.4, 102.7)
- moved R21 1.70 mm to (188.2, 111.6), turned to 0 degrees
- moved J6 1.55 mm to (202.4, 117.6)
- moved J4 1.27 mm to (179.7, 114.3)
- moved R5 0.13 mm to (124.3, 95.2)
Connections:
- J2 pad 2: /REF -> /1.5V
- J4 pad 2: /REF -> /1.5V
- R10 pad 2: /REF -> /1.5V
- R15 pad 2: /REF -> /1.5V
- R17 pad 2: /REF -> /1.5V
- R19 pad 1: /TEMP -> /PULSE
- R19 pad 2: Net-(U5A--) -> Net-(U5A-+)
- R2 pad 1: GND -> Net-(R2-Pad1)
- R20 pad 1: Net-(U5A--) -> Net-(U5A-+)
- R20 pad 2: /REF -> GND
- R21 pad 1: Net-(J5-Pin_1) -> /TEMP
- R3 pad 2: +5V -> /3V
- R5 pad 2: /PULSE -> Net-(U5A--)
- R7 pad 2: /REF -> /1.5V
- R9 pad 2: /REF -> /1.5V
- U2 pad 6: /REF -> /1.5V
- U2 pad 7: /REF -> /1.5V
- U5 pad 1: /TEMP -> Net-(U5A--)
- U5 pad 12: unconnected-(U5D-+-Pad12) -> Net-(U5D-+)
- U5 pad 13: unconnected-(U5D---Pad13) -> /3V
- U5 pad 14: unconnected-(U5-Pad14) -> /3V
- U5 pad 3: Net-(J5-Pin_1) -> Net-(U5A-+)
Routing:
- net /REF: track 149.7 -> 0.00 mm
- net /1.5V: track 0.00 -> 129.2 mm
- net /3V: track 0.00 -> 98.8 mm
- net Net-(U5A--): track 5.58 -> 100.1 mm
- net /PULSE: track 78.0 -> 24.2 mm
- net Net-(U5D-+): track 0.00 -> 47.4 mm
- net GND: track 225.9 -> 267.2 mm
- net +5V: track 179.4 -> 206.8 mm
- net Net-(U5A-+): track 0.00 -> 21.6 mm
- net /TEMP: track 41.9 -> 25.7 mm
- net Net-(J5-Pin_1): track 15.3 -> 0.00 mm
- net Net-(R2-Pad1): track 0.00 -> 12.5 mm
- net /RELAY: track 78.8 -> 89.4 mm
- net /PH: track 43.1 -> 51.1 mm
- net /COND_READ: track 35.7 -> 43.7 mm
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