File: Proyecto/MóduloElectrónico/Main board/Main board.kicad_pcb (KiCad board)
At the start: 2 copper layers, 99.7 x 59.7 mm, 11 parts

Commit message: Final
Parts:
- removed the REF** at (137.2, 87.6)
- removed the REF** at (85.7, 49.6)
- removed the REF** at (137.2, 73.0)
- removed the REF** at (118.7, 57.1)
- removed the REF** at (85.7, 85.8)
- removed the REF** at (55.9, 47.0)
- removed the REF** at (85.7, 67.9)
- removed the REF** at (121.3, 104.1)
- added D1: LED, LED_THT:LED_D1.8mm_W3.3mm_H2.4mm, F.Cu at (76.8, 58.1)
- added D2: LED, LED_THT:LED_D1.8mm_W3.3mm_H2.4mm, F.Cu at (80.6, 58.1)
- added D3: LED, LED_THT:LED_D1.8mm_W3.3mm_H2.4mm, F.Cu at (84.5, 58.1)
- added D4: LED, LED_THT:LED_D1.8mm_W3.3mm_H2.4mm, F.Cu at (88.3, 58.1)
- added G***: LOGO, custom_library:dasboot, F.Cu at (50.8, 61.6)
- added J1: Conn_01x02_Pin, Connector_Molex:Molex_KK-254_AE-6410-02A_1x02_P2.54mm_Vertical, F.Cu at (119.4, 52.7)
- added J2: Conn_01x03_Pin, Connector_Molex:Molex_KK-254_AE-6410-03A_1x03_P2.54mm_Vertical, F.Cu at (106.7, 52.7)
- added J3: Conn_01x03_Pin, Connector_Molex:Molex_KK-254_AE-6410-03A_1x03_P2.54mm_Vertical, F.Cu at (94.0, 52.7)
- added J4: Conn_01x02_Pin, Connector_Molex:Molex_KK-254_AE-6410-02A_1x02_P2.54mm_Vertical, F.Cu at (128.9, 52.7)
- added J5: Conn_01x05_Pin, Connector_Molex:Molex_KK-254_AE-6410-05A_1x05_P2.54mm_Vertical, F.Cu at (62.2, 52.7)
- added J6: Conn_01x06_Pin, Connector_PinHeader_2.54mm:PinHeader_1x06_P2.54mm_Vertical, F.Cu at (59.7, 72.4)
- added R1: 510, Resistor_THT:R_Axial_DIN0204_L3.6mm_D1.6mm_P2.54mm_Vertical, F.Cu at (76.8, 50.8)
- added R2: 510, Resistor_THT:R_Axial_DIN0204_L3.6mm_D1.6mm_P2.54mm_Vertical, F.Cu at (80.6, 50.8)
- added R3: 510, Resistor_THT:R_Axial_DIN0204_L3.6mm_D1.6mm_P2.54mm_Vertical, F.Cu at (84.5, 50.8)
- added R4: 510, Resistor_THT:R_Axial_DIN0204_L3.6mm_D1.6mm_P2.54mm_Vertical, F.Cu at (88.3, 50.9)
- added REF**: MountingHole_3.2mm_M3, MountingHole:MountingHole_3.2mm_M3, F.Cu at (45.7, 104.7)
- added U1: ~, custom_library:LoRa-V4-Heltec, F.Cu at (103.1, 87.9)
- added U2: ~, custom_library:mt-3608, F.Cu at (111.3, 86.2)
- added U3: ~, custom_library:mt-3608, F.Cu at (111.3, 68.9)
- added U4: ~, custom_library:mt-3608, F.Cu at (111.2, 52.0)
- added U5: ULN2003, Package_DIP:DIP-16_W7.62mm, F.Cu at (62.2, 69.2)
Routing:
- net GND: track 0.00 -> 273.4 mm
- net /MOTOR_5V: track 0.00 -> 148.0 mm
- net /MCU_5V: track 0.00 -> 146.1 mm
- net /SENSOR_COMM: track 0.00 -> 68.0 mm
- net Net-(J1-Pin_1): track 0.00 -> 66.5 mm
- net /ROTATION_INFO: track 0.00 -> 59.7 mm
- net /M3: track 0.00 -> 32.3 mm
- net /M2: track 0.00 -> 32.3 mm
- net /M1: track 0.00 -> 32.3 mm
- net /M0: track 0.00 -> 32.3 mm
- net /SENSOR_5V: track 0.00 -> 28.9 mm
- net Net-(D4-K): track 0.00 -> 28.7 mm
- net Net-(D3-K): track 0.00 -> 27.5 mm
- net Net-(D2-K): track 0.00 -> 26.2 mm
- net Net-(D1-K): track 0.00 -> 24.9 mm
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- added copper zone on B.Cu, net GND
- added copper zone on F.Cu, net GND
