File: Proyecto/MóduloElectrónico/Main board/Main board.kicad_sch (KiCad schematic)
At the start: 0 parts

Commit message: Final
Parts:
- added D1, D2, D3, D4: LED, LED_THT:LED_D1.8mm_W3.3mm_H2.4mm, symbol Device:LED
- added J1, J4: Conn_01x02_Pin, Connector_Molex:Molex_KK-254_AE-6410-02A_1x02_P2.54mm_Vertical, symbol Connector:Conn_01x02_Pin
- added J2, J3: Conn_01x03_Pin, Connector_Molex:Molex_KK-254_AE-6410-03A_1x03_P2.54mm_Vertical, symbol Connector:Conn_01x03_Pin
- added J5: Conn_01x05_Pin, Connector_Molex:Molex_KK-254_AE-6410-05A_1x05_P2.54mm_Vertical, symbol Connector:Conn_01x05_Pin
- added J6: Conn_01x06_Pin, Connector_PinHeader_2.54mm:PinHeader_1x06_P2.54mm_Vertical, symbol Connector:Conn_01x06_Pin
- added R1, R2, R3, R4: 510, Resistor_THT:R_Axial_DIN0204_L3.6mm_D1.6mm_P2.54mm_Vertical, symbol Device:R
- added U1: (no value), custom_library:LoRa-V4-Heltec, symbol Custom_library:LoRa
- added U2, U3, U4: (no value), custom_library:mt-3608, symbol Custom_library:MT3608
- added U5: ULN2003, Package_DIP:DIP-16_W7.62mm, symbol Transistor_Array:ULN2003
Connections:
- new net: D2.1 (K), J5.2 (Pin_2), U5.15 (O2)
- new net: D2.2 (A), R2.2
- new net: D4.1 (K), J5.4 (Pin_4), U5.13 (O4)
- new net: D4.2 (A), R4.2
- new net: J1.1 (Pin_1), U2.1 (VIN+), U3.1 (VIN+), U4.1 (VIN+)
- new net: J1.2 (Pin_2), J4.1 (Pin_1)
- new net: D3.2 (A), R3.2
- new net: D1.1 (K), J5.1 (Pin_1), U5.16 (O1)
- new net: D1.2 (A), R1.2
- new net: D3.1 (K), J5.3 (Pin_3), U5.14 (O3)
- new net GND: J2.3 (Pin_3), J3.3 (Pin_3), J4.2 (Pin_2), J6.6 (Pin_6), U1.1 (GND), U1.36 (GND), U2.2 (GND), U2.3 (GND), U3.2 (GND), U3.3 (GND), U4.2 (GND), U4.3 (GND), U5.8 (GND)
- new net M0: J6.2 (Pin_2), U1.9 (GPIO-36), U5.1 (I1)
- new net M1: J6.3 (Pin_3), U1.10 (GPIO-35), U5.2 (I2)
- new net M2: J6.4 (Pin_4), U1.11 (GPIO-34), U5.3 (I3)
- new net M3: J6.5 (Pin_5), U1.12 (GPIO-33), U5.4 (I4)
- new net MCU_5V: J3.1 (Pin_1), U1.2 (5V), U3.4 (VOUT+)
- new net MOTOR_5V: J5.5 (Pin_5), J6.1 (Pin_1), R1.1, R2.1, R3.1, R4.1, U2.4 (VOUT+), U5.9 (COM)
- new net ROTATION_INFO: J3.2 (Pin_2), U1.8 (GPIO-0)
- new net SENSOR_5V: J2.1 (Pin_1), U4.4 (VOUT+)
- new net SENSOR_COMM: J2.2 (Pin_2), U1.13 (GPIO-47)
- no-connect marks 0 -> 33
