File: Proyecto/MóduloElectrónico/Sensing probe - Alternate/Sensing probe.kicad_sch (KiCad schematic)
At the start: 46 parts, among them J1 Conn_01x02, J2 Conn_01x02, J3 Conn_01x03_Pin, J4 Conn_01x02, J5 Conn_01x03_Pin, J6 Conn_01x03_Pin, K1 HFD23, K2 HFD23, Q1 Q_NPN_EBC, U1 CA3140, U2 LM324, U4 CA3140, U5 LM324

Commit message: Final
Parts:
- R8: value 50K -> 15K
Changed lines of the file:
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@@
 			)
 		)
-		(property "Value" "50K"
+		(property "Value" "15K"
 			(at 135.89 138.684 90)
 			(show_name no)
