File: Proyecto/MóduloElectrónico/Esquemáticos KiCad/Main board/Main board.kicad_sch (KiCad schematic)
At the start: 20 parts, among them J1 Conn_01x02_Pin, J2 Conn_01x03_Pin, J3 Conn_01x03_Pin, J4 Conn_01x02_Pin, J5 Conn_01x05_Pin, J6 Conn_01x06_Pin, U5 ULN2003

Commit message: hola
Other:
- company: (none) -> Universidad Peruana Cayetano Heredia
- title: (none) -> Esquematico E04
